File: bolt-on-bosch-pst-f-1/Bolt-On Template.brd (EAGLE design)
At the start: 42 x 72 mm, 10 parts

Commit message: add labels to jst pins
Connections:
- net N$1 renamed PRESS_SIG
Changed lines of the file:
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@@
 <drawing>
 <settings>
-<setting alwaysvectorfont="yes"/>
+<setting alwaysvectorfont="no"/>
 <setting keepoldvectorfont="yes"/>
 <setting verticaltext="up"/>
@@
 <wire x1="26" y1="30" x2="26" y2="28" width="0.1524" layer="16"/>
 </signal>
-<signal name="N$1">
+<signal name="PRESS_SIG">
 <contactref element="R_PRESS_TOP" pad="2"/>
 <contactref element="PST-F_1_IN" pad="2"/>
